Commit message: simplified repo structure, add gazebo_ros export tags, fix gazebo_ros source dependency

File: urdf/simple_quad.urdf.xacro (robot description, xacro)
@@ -138,8 +138,4 @@
           <bias_mean>0.0000075</bias_mean>
           <bias_stddev>0.0000008</bias_stddev>
-          <!-- <mean>0.0</mean>
-          <stddev>0.0</stddev>
-          <bias_mean>0.0</bias_mean>
-          <bias_stddev>0.0</bias_stddev> -->
         </noise>
       </x>
@@ -150,8 +146,4 @@
           <bias_mean>0.0000075</bias_mean>
           <bias_stddev>0.0000008</bias_stddev>
-          <!-- <mean>0.0</mean>
-          <stddev>0.0</stddev>
-          <bias_mean>0.0</bias_mean>
-          <bias_stddev>0.0</bias_stddev> -->
         </noise>
       </y>
@@ -162,8 +154,4 @@
           <bias_mean>0.0000075</bias_mean>
           <bias_stddev>0.0000008</bias_stddev>
-          <!-- <mean>0.0</mean>
-          <stddev>0.0</stddev>
-          <bias_mean>0.0</bias_mean>
-          <bias_stddev>0.0</bias_stddev> -->
         </noise>
       </z>
@@ -176,8 +164,4 @@
           <bias_mean>0.1</bias_mean>
           <bias_stddev>0.001</bias_stddev>
-          <!-- <mean>0.0</mean>
-          <stddev>0.0</stddev>
-          <bias_mean>0.0</bias_mean>
-          <bias_stddev>0.0</bias_stddev> -->
         </noise>
       </x>
@@ -188,8 +172,4 @@
           <bias_mean>0.1</bias_mean>
           <bias_stddev>0.001</bias_stddev>
-          <!-- <mean>0.0</mean>
-          <stddev>0.0</stddev>
-          <bias_mean>0.0</bias_mean>
-          <bias_stddev>0.0</bias_stddev> -->
         </noise>
       </y>
@@ -200,8 +180,4 @@
           <bias_mean>0.1</bias_mean>
           <bias_stddev>0.001</bias_stddev>
-          <!-- <mean>0.0</mean>
-          <stddev>0.0</stddev>
-          <bias_mean>0.0</bias_mean>
-          <bias_stddev>0.0</bias_stddev> -->
         </noise>
       </z>
@@ -210,5 +186,5 @@
 </sensor>
 </gazebo>
-<link name="lidar_link">
+<!-- <link name="lidar_link">
   <inertial>
     <origin xyz="0 0 0" rpy="0 0 0"/>
@@ -233,9 +209,9 @@
   <child link="lidar_link"/>
   <origin xyz="0 0 ${base_height}" rpy="0 0 0"/>
-</joint>
-<gazebo reference="lidar_link">
-  <sensor name="lidar" type="ray">
+</joint> -->
+<!-- <gazebo reference="lidar_link">
+  <sensor name="lidar" type="gpu_ray">
     <always_on>true</always_on>
-    <visualize>true</visualize>
+    <visualize>false</visualize>
     <update_rate>5</update_rate>
     <ray>
@@ -268,5 +244,5 @@
     </plugin>
   </sensor>
-</gazebo>
+</gazebo> -->
 <link name="camera_link">
   <visual>
@@ -361,5 +337,5 @@
     <update_rate>50</update_rate>
     <publish_odom>true</publish_odom>
-    <publish_odom_tf>false</publish_odom_tf>
+    <publish_odom_tf>true</publish_odom_tf>
     <cmd_vel_topic>/cmd_vel</cmd_vel_topic>
     <cmd_pos_topic>/cmd_pos</cmd_pos_topic>
